Commit message: tape localization WIP

File: urdf/turtlebot3_waffle_pi.gazebo.xacro (robot description, xacro)
@@ -140,5 +140,5 @@
       <visualize>$(arg camera_visual)</visualize>
       <camera>
-          <horizontal_fov>1.085595</horizontal_fov>
+          <horizontal_fov>1.2</horizontal_fov>
           <image>
               <width>640</width>

File: urdf/turtlebot3_waffle_pi.urdf.xacro (robot description, xacro)
@@ -2,5 +2,5 @@
 <robot name="turtlebot3_waffle_pi" xmlns:xacro="http://ros.org/wiki/xacro">
   <xacro:include filename="$(find turtlebot3_description)/urdf/common_properties.xacro"/>
-  <xacro:include filename="$(find turtlebot3_description)/urdf/turtlebot3_waffle_pi.gazebo.xacro"/>
+  <xacro:include filename="$(find grid_nav)/urdf/turtlebot3_waffle_pi.gazebo.xacro"/>
   <link name="base_footprint"/>
   <joint name="base_joint" type="fixed">
@@ -174,5 +174,5 @@
   </link>
   <joint name="camera_rgb_joint" type="fixed">
-    <origin xyz="0.003 0.011 0.009" rpy="0 0 0"/>
+    <origin xyz="0.1 0.011 0.3" rpy="0 1.57 0"/>
     <parent link="camera_link"/>
     <child link="camera_rgb_frame"/>
